Commit message: cleanup for ROS1/ROS2

File: urdf/ECM.urdf.xacro (robot description, xacro)
@@ -2,5 +2,5 @@
 <robot name="ecm" xmlns:xacro="http://www.ros.org/wiki/xacro">
   <!-- Macros -->
-  <xacro:include filename="$(find dvrk_model)/model/ecm.urdf.xacro"/>
+  <xacro:include filename="$(find dvrk_model)/urdf/ecm.urdf.xacro"/>
   <link name="world"/>
   <xacro:ecm

File: urdf/MTML.urdf.xacro (robot description, xacro)
@@ -2,9 +2,9 @@
 <robot name="master" xmlns:xacro="http://www.ros.org/wiki/xacro">
   <!-- Macros -->
-  <xacro:include filename="$(find dvrk_model)/model/mtm.urdf.xacro"/>
+  <xacro:include filename="$(find dvrk_model)/urdf/mtm.urdf.xacro"/>
   <link name="world"/>
-  <xacro:mtm_right
-      prefix="MTMR_"
+  <xacro:mtm_left
+      prefix="MTML_"
       parent_link="world"
-      xyz="0.25 0.0 1.0" rpy="0.0 0.0 0.0"/>
+      xyz="-0.25 0.0 1.0" rpy="0.0 0.0 0.0"/>
 </robot>

File: urdf/MTMR.urdf.xacro (robot description, xacro)
@@ -2,9 +2,9 @@
 <robot name="master" xmlns:xacro="http://www.ros.org/wiki/xacro">
   <!-- Macros -->
-  <xacro:include filename="$(find dvrk_model)/model/mtm.urdf.xacro"/>
+  <xacro:include filename="$(find dvrk_model)/urdf/mtm.urdf.xacro"/>
   <link name="world"/>
-  <xacro:mtm_left
-      prefix="MTML_"
+  <xacro:mtm_right
+      prefix="MTMR_"
       parent_link="world"
-      xyz="-0.25 0.0 1.0" rpy="0.0 0.0 0.0"/>
+      xyz="0.25 0.0 1.0" rpy="0.0 0.0 0.0"/>
 </robot>

File: urdf/PSM1_Snake.urdf.xacro (robot description, xacro)
@@ -2,9 +2,9 @@
 <robot name="dvrk_psm" xmlns:xacro="http://www.ros.org/wiki/xacro">
   <!-- Macros -->
-  <xacro:include filename="$(find dvrk_model)/model/psm.urdf.xacro"/>
+  <xacro:include filename="$(find dvrk_model)/urdf/psm.urdf.xacro"/>
   <link name="world"/>
-  <xacro:psm_caudier
-      prefix="PSM2_"
+  <xacro:psm_snake
+      prefix="$(arg prefix)"
       parent_link="world"
-      xyz="0.25 0.0 0.5" rpy="0.0 0.0 -3.1415926"/>
+      xyz="-0.25 0.0 0.5" rpy="0.0 0.0 3.1415926"/>
 </robot>

File: urdf/PSM2.urdf.xacro (robot description, xacro)
@@ -2,9 +2,9 @@
 <robot name="dvrk_psm" xmlns:xacro="http://www.ros.org/wiki/xacro">
   <!-- Macros -->
-  <xacro:include filename="$(find dvrk_model)/model/psm.urdf.xacro"/>
+  <xacro:include filename="$(find dvrk_model)/urdf/psm.urdf.xacro"/>
   <link name="world"/>
-  <xacro:psm_sca
-      prefix="PSM1_"
+  <xacro:psm_caudier
+      prefix="PSM2_"
       parent_link="world"
-      xyz="-0.25 0.0 0.5" rpy="0.0 0.0 3.1415926"/>
+      xyz="0.25 0.0 0.5" rpy="0.0 0.0 -3.1415926"/>
 </robot>

File: urdf/PSM3.urdf.xacro (robot description, xacro)
@@ -2,9 +2,9 @@
 <robot name="dvrk_psm" xmlns:xacro="http://www.ros.org/wiki/xacro">
   <!-- Macros -->
-  <xacro:include filename="$(find dvrk_model)/model/psm.urdf.xacro"/>
+  <xacro:include filename="$(find dvrk_model)/urdf/psm.urdf.xacro"/>
   <link name="world"/>
-  <xacro:psm_snake
+  <xacro:psm_caudier
       prefix="$(arg prefix)"
       parent_link="world"
-      xyz="-0.25 0.0 0.5" rpy="0.0 0.0 3.1415926"/>
+      xyz="0.50 0.0 0.5" rpy="0.0 0.0 -3.1415926"/>
 </robot>

File: urdf/both_psms.urdf.xacro (robot description, xacro)
@@ -2,15 +2,15 @@
 <robot name="dvrk_psm" xmlns:xacro="http://www.ros.org/wiki/xacro">
   <!-- Macros -->
-  <xacro:include filename="$(find dvrk_model)/model/psm.urdf.xacro"/>
+  <xacro:include filename="$(find dvrk_model)/urdf/psm.urdf.xacro"/>
   <link name="world">
-      <origin xyz="0.0 0.0 0.0"/>
+    <origin xyz="0.0 0.0 0.0"/>
   </link>
   <joint name="world_joint" type="fixed">
-      <parent link="world"/>
-      <child link="camera"/>
-      <origin rpy="0.0 0.0 0.0" xyz="0.0 0.0 0.0"/>
+    <parent link="world"/>
+    <child link="camera"/>
+    <origin rpy="0.0 0.0 0.0" xyz="0.0 0.0 0.0"/>
   </joint>
   <link name="camera">
-  <origin rpy="0.0 0.0 0.0" xyz="0.0 0.2 0.8"/>
+    <origin rpy="0.0 0.0 0.0" xyz="0.0 0.2 0.8"/>
   </link>
   <xacro:psm

File: urdf/ecm.urdf.xacro (robot description, xacro)
@@ -2,5 +2,5 @@
 <robot name="ecm" xmlns:xacro="http://www.ros.org/wiki/xacro">
   <!-- Colors -->
-  <xacro:include filename="$(find dvrk_model)/model/common.urdf.xacro"/>
+  <xacro:include filename="$(find dvrk_model)/urdf/common.urdf.xacro"/>
   <!-- Macro for da Vinci Endoscope Camera Manipulator (ECM) -->
   <xacro:macro name="ecm" params="prefix parent_link xyz rpy">

File: urdf/mtm.urdf.xacro (robot description, xacro)
@@ -2,5 +2,5 @@
 <robot name="mtm" xmlns:xacro="http://www.ros.org/wiki/xacro">
   <!-- Colors -->
-  <xacro:include filename="$(find dvrk_model)/model/common.urdf.xacro"/>
+  <xacro:include filename="$(find dvrk_model)/urdf/common.urdf.xacro"/>
   <!-- Macro for the da Vinci Master Console -->
   <xacro:macro name="master_console" params="prefix parent_link xyz rpy">
@@ -24,7 +24,7 @@
   <xacro:macro name="mtm_right" params="prefix parent_link xyz rpy">
     <xacro:mtm
-      prefix="${prefix}"
-      parent_link="${parent_link}"
-      xyz="${xyz}" rpy="${rpy}"/>
+	prefix="${prefix}"
+	parent_link="${parent_link}"
+	xyz="${xyz}" rpy="${rpy}"/>
     <xacro:mtm_platform_right prefix="${prefix}"/>
   </xacro:macro>
@@ -54,6 +54,6 @@
         <mass value=".9"/>
         <inertia ixx="9.0" ixy="0.0" ixz="0.0"
-                           iyy="9.0" iyz="0.0"
-                                     izz="9.0"/>
+                 iyy="9.0" iyz="0.0"
+                 izz="9.0"/>
       </inertial>
     </link>

File: urdf/psm.tool.sca.urdf.xacro (robot description, xacro)
@@ -2,5 +2,5 @@
 <robot name="dvrk_psm" xmlns:xacro="http://www.ros.org/wiki/xacro">
   <!-- This file contains different tool urdf -->
-  <xacro:include filename="$(find dvrk_model)/model/common.urdf.xacro"/>
+  <xacro:include filename="$(find dvrk_model)/urdf/common.urdf.xacro"/>
   <!-- sca  -->
   <xacro:macro name="psm_tool_sca" params="prefix">

File: urdf/psm.urdf.xacro (robot description, xacro)
@@ -2,8 +2,8 @@
 <robot name="dvrk_psm" xmlns:xacro="http://www.ros.org/wiki/xacro">
   <!-- Macros -->
-  <xacro:include filename="$(find dvrk_model)/model/psm.base.urdf.xacro"/>
-  <xacro:include filename="$(find dvrk_model)/model/psm.tool.sca.urdf.xacro"/>
-  <xacro:include filename="$(find dvrk_model)/model/psm.tool.caudier.urdf.xacro"/>
-  <xacro:include filename="$(find dvrk_model)/model/psm.tool.snake.urdf.xacro"/>
+  <xacro:include filename="$(find dvrk_model)/urdf/psm.base.urdf.xacro"/>
+  <xacro:include filename="$(find dvrk_model)/urdf/psm.tool.sca.urdf.xacro"/>
+  <xacro:include filename="$(find dvrk_model)/urdf/psm.tool.caudier.urdf.xacro"/>
+  <xacro:include filename="$(find dvrk_model)/urdf/psm.tool.snake.urdf.xacro"/>
   <!-- Macro for psm with snake -->
   <xacro:macro name="psm_snake" params="prefix parent_link xyz rpy">
