Commit message: Removed useless outer_ prefix from joint names

File: urdf/ecm.urdf.xacro (robot description, xacro)
@@ -41,5 +41,5 @@
     <link name="${prefix}_base_link"/>
     <!-- Joint 1: Outer Yaw -->
-    <joint name="outer_yaw" type="revolute">
+    <joint name="yaw" type="revolute">
       <parent link="${prefix}_base_link"/>
       <child link="${prefix}_yaw_link"/>
@@ -67,5 +67,5 @@
     </link>
     <!-- Joint 2: Pitch -->
-    <joint name="outer_pitch" type="revolute">
+    <joint name="pitch" type="revolute">
       <parent link="${prefix}_yaw_link"/>
       <child link="${prefix}_pitch_link"/>
@@ -76,5 +76,5 @@
     </joint>
     <link name="${prefix}_pitch_link"/>
-    <joint name="outer_pitch_0" type="continuous">
+    <joint name="pitch_0" type="continuous">
       <parent link="${prefix}_yaw_link"/>
       <child link="${prefix}_pitch_link_1"/>
@@ -82,5 +82,5 @@
       <axis xyz="0 0 1"/>
       <joint_properties damping="1.0" friction="0.0"/>
-      <mimic joint="outer_pitch" multiplier="1"/>
+      <mimic joint="pitch" multiplier="1"/>
     </joint>
     <link name="${prefix}_pitch_link_1">
@@ -103,5 +103,5 @@
       </inertial>
     </link>
-    <joint name="outer_pitch_1" type="continuous">
+    <joint name="pitch_1" type="continuous">
       <parent link="${prefix}_pitch_link_1"/>
       <child link="${prefix}_pitch_link_2"/>
@@ -109,5 +109,5 @@
       <axis xyz="0 0 1"/>
       <joint_properties damping="1.0" friction="0.0"/>
-      <mimic joint="outer_pitch" multiplier="-1"/>
+      <mimic joint="pitch" multiplier="-1"/>
     </joint>
     <link name="${prefix}_pitch_link_2">
@@ -130,5 +130,5 @@
       </inertial>
     </link>
-    <joint name="outer_pitch_2" type="continuous">
+    <joint name="pitch_2" type="continuous">
       <parent link="${prefix}_pitch_link_2"/>
       <child link="${prefix}_pitch_link_3"/>
@@ -136,5 +136,5 @@
       <axis xyz="0 0 1"/>
       <joint_properties damping="1.0" friction="0.0"/>
-      <mimic joint="outer_pitch" multiplier="1"/>
+      <mimic joint="pitch" multiplier="1"/>
     </joint>
     <link name="${prefix}_pitch_link_3">
@@ -182,5 +182,5 @@
     </link>
     <!-- Joint 4: Roll -->
-    <joint name="outer_roll" type="revolute">
+    <joint name="roll" type="revolute">
       <parent link="${prefix}_insertion_link"/>
       <child link="${prefix}_roll_link"/>

File: urdf/psm.base.urdf.xacro (robot description, xacro)
@@ -18,5 +18,5 @@
     </link>
     <!-- joint 1 -->
-    <joint name="outer_yaw" type="revolute">
+    <joint name="yaw" type="revolute">
       <parent link="${prefix}psm_base_link"/>
       <child link="${prefix}outer_yaw_link"/>
@@ -39,5 +39,5 @@
     <!-- link, all visual links mimic outer_pitch value -->
     <!-- joint 2: outer_pitch -->
-    <joint name="outer_pitch" type="revolute">
+    <joint name="pitch" type="revolute">
       <parent link="${prefix}outer_yaw_link"/>
       <child link="${prefix}outer_pitch_link"/>
@@ -49,5 +49,5 @@
     <link name="${prefix}outer_pitch_link"/>
     <!-- joint 2-1: outer_pitch_1 -->
-    <joint name="outer_pitch_1" type="continuous">
+    <joint name="pitch_1" type="continuous">
       <parent link="${prefix}outer_yaw_link"/>
       <child link="${prefix}outer_pitch_back_link"/>
@@ -55,5 +55,5 @@
       <!-- <origin rpy="-1.5708 -1.5708 0" xyz="0 0.0295 0.1495"/> -->
       <origin rpy="-1.5708 -1.5708 0" xyz="0 0.0295 0.5185"/>
-      <mimic joint="outer_pitch" multiplier="1"/>
+      <mimic joint="pitch" multiplier="1"/>
     </joint>
     <!-- link 2-1: outer_pitch_back -->
@@ -67,10 +67,10 @@
     </link>
     <!-- joint 2-2: outer_pitch_2 -->
-    <joint name="outer_pitch_2" type="continuous">
+    <joint name="pitch_2" type="continuous">
       <parent link="${prefix}outer_yaw_link"/>
       <child link="${prefix}outer_pitch_front_link"/>
       <axis xyz="0 0 1"/>
       <origin rpy="-1.5708 -1.5708 0" xyz="0 0.0295 0.4285"/>
-      <mimic joint="outer_pitch" multiplier="1"/>
+      <mimic joint="pitch" multiplier="1"/>
     </joint>
     <!-- link 2-2: outer_pitch_front -->
@@ -84,10 +84,10 @@
     </link>
     <!-- joint 2-3: outer_pitch_3 -->
-    <joint name="outer_pitch_3" type="continuous">
+    <joint name="pitch_3" type="continuous">
       <parent link="${prefix}outer_pitch_back_link"/>
       <child link="${prefix}outer_pitch_bottom_link"/>
       <axis xyz="0 0 1"/>
       <origin rpy="0 0 0" xyz="0.04178 0.15007 -0.0137"/>
-      <mimic joint="outer_pitch" multiplier="-1"/>
+      <mimic joint="pitch" multiplier="-1"/>
     </joint>
     <!-- link 2-3: outer_pitch_bottom -->
@@ -101,10 +101,10 @@
     </link>
     <!-- joint 2-4: outer_pitch_4 -->
-    <joint name="outer_pitch_4" type="continuous">
+    <joint name="pitch_4" type="continuous">
       <parent link="${prefix}outer_pitch_back_link"/>
       <child link="${prefix}outer_pitch_top_link"/>
       <axis xyz="0 0 1"/>
       <origin rpy="0 0 0" xyz="0.04209 0.18695 -0.02412"/>
-      <mimic joint="outer_pitch" multiplier="-1"/>
+      <mimic joint="pitch" multiplier="-1"/>
     </joint>
     <!-- link 2-4: outer_pitch_top -->
@@ -118,10 +118,10 @@
     </link>
     <!-- joint 2-5: outer_pitch_5 -->
-    <joint name="outer_pitch_5" type="continuous">
+    <joint name="pitch_5" type="continuous">
       <parent link="${prefix}outer_pitch_bottom_link"/>
       <child link="${prefix}outer_insertion_link"/>
       <axis xyz="0 0 1"/>
       <origin rpy="0 0 0" xyz="-0.520 0 -0.0155"/>
-      <mimic joint="outer_pitch" multiplier="1"/>
+      <mimic joint="pitch" multiplier="1"/>
     </joint>
     <!-- link 2-5: outer_insertion -->
@@ -135,5 +135,5 @@
     </link>
     <!-- joint 3: insertion -->
-    <joint name="outer_insertion" type="prismatic">
+    <joint name="insertion" type="prismatic">
       <!-- <parent link="${prefix}outer_insertion_link"/> -->
       <!-- <parent link="${prefix}psm_base_link"/> -->
@@ -154,5 +154,5 @@
     </link>
     <!-- joint 4: Outer Roll -->
-    <joint name="outer_roll" type="revolute">
+    <joint name="roll" type="revolute">
       <parent link="${prefix}tool_main_link"/>
       <child link="${prefix}tool_wrist_link"/>
@@ -171,5 +171,5 @@
     </link>
     <!-- joint 4-1: outer roll shaft joint FIXED-->
-    <joint name="outer_roll_shaft" type="fixed">
+    <joint name="roll_shaft" type="fixed">
       <parent link="${prefix}tool_wrist_link"/>
       <child link="${prefix}tool_wrist_shaft_link"/>

File: urdf/psm.tool.caudier.urdf.xacro (robot description, xacro)
@@ -3,5 +3,5 @@
   <xacro:macro name="psm_tool_caudier" params="prefix">
     <!-- joint 5: Outer wrist pitch joint -->
-    <joint name="outer_wrist_pitch" type="revolute">
+    <joint name="wrist_pitch" type="revolute">
       <parent link="${prefix}tool_wrist_shaft_link"/>
       <child link="${prefix}tool_wrist_caudier_link"/>
@@ -27,5 +27,5 @@
     </link>
     <!-- joint 6: Tool wrist yaw joint -->
-    <joint name="outer_wrist_yaw" type="revolute">
+    <joint name="wrist_yaw" type="revolute">
       <parent link="${prefix}tool_wrist_caudier_link"/>
       <child link="${prefix}tool_wrist_caudier_link_shaft"/>

File: urdf/psm.tool.sca.urdf.xacro (robot description, xacro)
@@ -6,5 +6,5 @@
   <xacro:macro name="psm_tool_sca" params="prefix">
     <!-- joint 5: Outer wrist pitch joint -->
-    <joint name="outer_wrist_pitch" type="revolute">
+    <joint name="wrist_pitch" type="revolute">
       <parent link="${prefix}tool_wrist_shaft_link"/>
       <child link="${prefix}tool_wrist_sca_link"/>
@@ -24,5 +24,5 @@
     </link>
     <!-- joint 6: Outer wrist yaw joint -->
-    <joint name="outer_wrist_yaw" type="revolute">
+    <joint name="wrist_yaw" type="revolute">
       <parent link="${prefix}tool_wrist_sca_link"/>
       <child link="${prefix}tool_wrist_sca_shaft_link"/>

File: urdf/psm.tool.snake.urdf.xacro (robot description, xacro)
@@ -4,5 +4,5 @@
   <xacro:macro name="psm_tool_snake" params="prefix">
     <!-- joint 6: Outer wrist pitch1 joint -->
-    <joint name="outer_wrist_pitch1" type="revolute">
+    <joint name="wrist_pitch1" type="revolute">
       <parent link="${prefix}tool_wrist_shaft_link"/>
       <child link="${prefix}tool_snake_disc1_link"/>
@@ -21,5 +21,5 @@
     </link>
     <!-- joint 7: Outer wrist yaw1 joint -->
-    <joint name="outer_wrist_yaw1" type="revolute">
+    <joint name="wrist_yaw1" type="revolute">
       <parent link="${prefix}tool_snake_disc1_link"/>
       <child link="${prefix}tool_snake_disc2_link"/>
@@ -38,5 +38,5 @@
     </link>
     <!-- joint 8: Outer wrist yaw2 joint -->
-    <joint name="outer_wrist_yaw2" type="revolute">
+    <joint name="wrist_yaw2" type="revolute">
       <parent link="${prefix}tool_snake_disc2_link"/>
       <child link="${prefix}tool_snake_disc3_link"/>
@@ -55,5 +55,5 @@
     </link>
     <!-- joint 9: Outer wrist pitch2 joint -->
-    <joint name="outer_wrist_pitch2" type="revolute">
+    <joint name="wrist_pitch2" type="revolute">
       <parent link="${prefix}tool_snake_disc3_link"/>
       <child link="${prefix}tool_snake_end_link"/>
